Commit message: 가제보 월드 +f110 스폰

File: f110_description/urdf/f1tenth.urdf.xacro (robot description, xacro)
@@ -5,5 +5,7 @@
 Vehicle: Traxxas Fiesta ST Rally 1/10 Scale
 -->
-<robot name="f1tenth_racecar">
+<robot name="f1tenth_racecar" xmlns:xacro="http://www.ros.org/wiki/xacro">
+  <!-- Include Hokuyo LiDAR -->
+  <xacro:include filename="$(find f110_description)/urdf/hokuyo.urdf.xacro"/>
   <!-- ============================================ -->
   <!-- Materials -->
@@ -37,42 +39,26 @@
       <material name="blue"/>
     </visual>
-    <!-- 바퀴와의 간섭을 없기 위함
     <collision>
       <origin xyz="0.165 0 0.09" rpy="0 0 0"/>
       <geometry>
-        <box size="0.3302 0.2032 0.1"/>
-      </geometry>
-    </collision>
-    -->
+        <box size="0.05 0.001 0.006"/>  <!-- Very small to avoid wheel collision -->
+      </geometry>
+    </collision>
   </link>
   <!-- ============================================ -->
   <!-- LiDAR (Hokuyo 10LX) -->
   <!-- ============================================ -->
-  <joint name="base_to_laser" type="fixed">
-    <parent link="base_link"/>
-    <child link="laser"/>
-    <origin xyz="0.275 0 0.19" rpy="0 0 0"/>  <!-- 0.275m forward, 0.19m high -->
-  </joint>
-  <link name="laser">
-    <inertial>
-      <mass value="0.130"/>  <!-- Hokuyo 10LX actual mass -->
-      <origin xyz="0 0 0" rpy="0 0 0"/>
-      <inertia
-        ixx="0.0001" ixy="0.0" ixz="0.0"
-        iyy="0.0001" iyz="0.0"
-        izz="0.0001"/>
-    </inertial>
-    <visual>
-      <geometry>
-        <cylinder radius="0.026" length="0.05"/>
-      </geometry>
-      <material name="black"/>
-    </visual>
-    <collision>
-      <geometry>
-        <cylinder radius="0.026" length="0.05"/>
-      </geometry>
-    </collision>
-  </link>
+  <xacro:hokuyo_10lx
+    parent="base_link"
+    name="laser"
+    topic="/scan"
+    hz="10"
+    samples="1080"
+    min_angle="-2.35619"
+    max_angle="2.35619"
+    min_range="0.1"
+    max_range="30.0">
+    <origin xyz="0.275 0 0.19" rpy="0 0 0"/>
+  </xacro:hokuyo_10lx>
   <!-- ============================================ -->
   <!-- IMU Sensor -->
@@ -100,14 +86,48 @@
     </collision>
   </link>
+  <!-- Gazebo IMU Sensor -->
+  <gazebo reference="imu_link">
+    <sensor name="imu_sensor" type="imu">
+      <always_on>true</always_on>
+      <update_rate>100</update_rate>
+      <plugin filename="libgazebo_ros_imu_sensor.so" name="imu_plugin">
+        <ros>
+          <namespace>/f1tenth</namespace>
+          <remapping>~/out:=imu</remapping>
+        </ros>
+        <initial_orientation_as_reference>false</initial_orientation_as_reference>
+      </plugin>
+    </sensor>
+  </gazebo>
+  <!-- ============================================ -->
+  <!-- Steering Wheel (dummy joint for Ackermann plugin) -->
+  <!-- ============================================ -->
+  <joint name="steering_wheel_joint" type="revolute">
+    <parent link="base_link"/>
+    <child link="steering_wheel_link"/>
+    <origin xyz="0.15 0 0.25" rpy="0 0 0"/>
+    <axis xyz="0 0 1"/>
+    <limit lower="-6.283" upper="6.283" effort="5.0" velocity="4.0"/>
+  </joint>
+  <link name="steering_wheel_link">
+    <inertial>
+      <mass value="0.01"/>
+      <origin xyz="0 0 0" rpy="0 0 0"/>
+      <inertia
+        ixx="1e-5" ixy="0.0" ixz="0.0"
+        iyy="1e-5" iyz="0.0"
+        izz="1e-5"/>
+    </inertial>
+  </link>
   <!-- ============================================ -->
   <!-- Rear Wheels (Fixed, Motor Controlled) -->
   <!-- ============================================ -->
   <!-- Left Rear Wheel -->
-  <joint name="left_rear_wheel_joint" type="revolute">
+  <joint name="left_rear_wheel_joint" type="continuous">
     <parent link="base_link"/>
     <child link="left_rear_wheel"/>
     <origin xyz="0 0.12065 0.0508" rpy="0 0 0"/>  <!-- y = (wheel_width + width)/2 -->
     <axis xyz="0 1 0"/>  <!-- Rotation around Y axis -->
-    <limit lower="-1e9" upper="1e9" effort="100.0" velocity="400.0"/>  <!-- VESC motor: 100 N·m -->
+    <dynamics damping="0.1" friction="0.1"/>
   </joint>
   <link name="left_rear_wheel">
@@ -138,10 +158,10 @@
   </link>
   <!-- Right Rear Wheel -->
-  <joint name="right_rear_wheel_joint" type="revolute">
+  <joint name="right_rear_wheel_joint" type="continuous">
     <parent link="base_link"/>
     <child link="right_rear_wheel"/>
     <origin xyz="0 -0.12065 0.0508" rpy="0 0 0"/>
     <axis xyz="0 1 0"/>
-    <limit lower="-1e9" upper="1e9" effort="100.0" velocity="400.0"/>  <!-- VESC motor: 100 N·m -->
+    <dynamics damping="0.1" friction="0.1"/>
   </joint>
   <link name="right_rear_wheel">
@@ -181,4 +201,5 @@
     <axis xyz="0 0 1"/>  <!-- Steering axis (vertical) -->
     <limit lower="-0.4189" upper="0.4189" effort="10.0" velocity="3.2"/>  <!-- ±24°, from F1TENTH Gym -->
+    <dynamics damping="0.7" friction="0.5"/>
   </joint>
   <link name="left_steering_hinge">
@@ -193,10 +214,10 @@
   </link>
   <!-- Left Front Wheel -->
-  <joint name="left_front_wheel_joint" type="revolute">
+  <joint name="left_front_wheel_joint" type="continuous">
     <parent link="left_steering_hinge"/>
     <child link="left_front_wheel"/>
     <origin xyz="0 0 0" rpy="0 0 0"/>
     <axis xyz="0 1 0"/>
-    <limit lower="-1e9" upper="1e9" effort="100.0" velocity="400.0"/>  <!-- AWD: VESC motor -->
+    <dynamics damping="0.1" friction="0.1"/>
   </joint>
   <link name="left_front_wheel">
@@ -233,4 +254,5 @@
     <axis xyz="0 0 1"/>
     <limit lower="-0.4189" upper="0.4189" effort="10.0" velocity="3.2"/>
+    <dynamics damping="0.7" friction="0.5"/>
   </joint>
   <link name="right_steering_hinge">
@@ -245,10 +267,10 @@
   </link>
   <!-- Right Front Wheel -->
-  <joint name="right_front_wheel_joint" type="revolute">
+  <joint name="right_front_wheel_joint" type="continuous">
     <parent link="right_steering_hinge"/>
     <child link="right_front_wheel"/>
     <origin xyz="0 0 0" rpy="0 0 0"/>
     <axis xyz="0 1 0"/>
-    <limit lower="-1e9" upper="1e9" effort="100.0" velocity="400.0"/>  <!-- AWD: VESC motor -->
+    <dynamics damping="0.1" friction="0.1"/>
   </joint>
   <link name="right_front_wheel">
@@ -278,38 +300,51 @@
     </collision>
   </link>
-  <gazebo reference="laser">
-    <sensor type="ray" name="hokuyo_sensor">
-      <pose>0 0 0 0 0 0</pose>
-      <visualize>false</visualize>
-      <update_rate>10</update_rate>
-      <ray>
-        <scan>
-          <horizontal>
-            <samples>1080</samples>
-            <resolution>1</resolution>
-            <min_angle>-2.35619</min_angle>
-            <max_angle>2.35619</max_angle>
-          </horizontal>
-        </scan>
-        <range>
-          <min>0.1</min>
-          <max>30.0</max>
-          <resolution>0.01</resolution>
-        </range>
-        <noise>
-          <type>gaussian</type>
-          <mean>0.0</mean>
-          <stddev>0.01</stddev>
-        </noise>
-      </ray>
-      <plugin name="gazebo_ros_ray_sensor" filename="libgazebo_ros_ray_sensor.so">
-        <ros>
-          <remapping>~/out:=/scan</remapping>
-        </ros>
-        <output_type>sensor_msgs/LaserScan</output_type>
-        <frame_name>laser</frame_name>
-      </plugin>
-    </sensor>
-  </gazebo>
+  <!-- Friction and contact parameters for base_link -->
+  <gazebo reference="base_link">
+    <mu1>0.1</mu1>
+    <mu2>0.1</mu2>
+    <kp>1000000.0</kp>
+    <kd>100.0</kd>
+    <material>Gazebo/Blue</material>
+    <self_collide>false</self_collide>
+  </gazebo>
+  <!-- Friction parameters for wheels -->
+  <gazebo reference="left_rear_wheel">
+    <mu1>1.5</mu1>
+    <mu2>1.5</mu2>
+    <kp>10000000.0</kp>
+    <kd>1.0</kd>
+    <minDepth>0.005</minDepth>
+    <maxVel>0.1</maxVel>
+    <self_collide>false</self_collide>
+  </gazebo>
+  <gazebo reference="right_rear_wheel">
+    <mu1>1.5</mu1>
+    <mu2>1.5</mu2>
+    <kp>10000000.0</kp>
+    <kd>1.0</kd>
+    <minDepth>0.005</minDepth>
+    <maxVel>0.1</maxVel>
+    <self_collide>false</self_collide>
+  </gazebo>
+  <gazebo reference="left_front_wheel">
+    <mu1>1.5</mu1>
+    <mu2>1.5</mu2>
+    <kp>10000000.0</kp>
+    <kd>1.0</kd>
+    <minDepth>0.005</minDepth>
+    <maxVel>0.1</maxVel>
+    <self_collide>false</self_collide>
+  </gazebo>
+  <gazebo reference="right_front_wheel">
+    <mu1>1.5</mu1>
+    <mu2>1.5</mu2>
+    <kp>10000000.0</kp>
+    <kd>1.0</kd>
+    <minDepth>0.005</minDepth>
+    <maxVel>0.1</maxVel>
+    <self_collide>false</self_collide>
+  </gazebo>
+  <!-- Ackermann Drive Controller Plugin -->
   <gazebo>
     <plugin name="gazebo_ros_ackermann_drive" filename="libgazebo_ros_ackermann_drive.so">
@@ -318,32 +353,39 @@
         <remapping>cmd_vel:=cmd_vel</remapping>
         <remapping>odom:=odom</remapping>
-        <remapping>distance:=distance</remapping>
       </ros>
       <update_rate>100.0</update_rate>
-      <front_left_joint>left_steering_hinge_joint</front_left_joint>
-      <front_right_joint>right_steering_hinge_joint</front_right_joint>
+      <!-- 바퀴 조인트 (회전) -->
+      <front_left_joint>left_front_wheel_joint</front_left_joint>
+      <front_right_joint>right_front_wheel_joint</front_right_joint>
       <rear_left_joint>left_rear_wheel_joint</rear_left_joint>
       <rear_right_joint>right_rear_wheel_joint</rear_right_joint>
+      <!-- 조향 조인트 -->
       <left_steering_joint>left_steering_hinge_joint</left_steering_joint>
       <right_steering_joint>right_steering_hinge_joint</right_steering_joint>
-      <steering_wheel_radius>0.0508</steering_wheel_radius>
+      <!-- 핵심: steering_wheel_joint 추가 (필수!) -->
+      <steering_wheel_joint>steering_wheel_joint</steering_wheel_joint>
+      <!-- PID Gains 추가 (안정성 향상) -->
+      <left_steering_pid_gain>1500 0 1</left_steering_pid_gain>
+      <left_steering_i_range>0 0</left_steering_i_range>
+      <right_steering_pid_gain>1500 0 1</right_steering_pid_gain>
+      <right_steering_i_range>0 0</right_steering_i_range>
+      <linear_velocity_pid_gain>1000 0 1</linear_velocity_pid_gain>
+      <linear_velocity_i_range>0 0</linear_velocity_i_range>
+      <!-- 조향 제한 -->
       <max_steer>0.4189</max_steer>
       <max_steering_angle>7.85</max_steering_angle>
-      <max_speed>20.0</max_speed>
-      <left_rear_wheel_spinning_joint>left_rear_wheel_joint</left_rear_wheel_spinning_joint>
-      <right_rear_wheel_spinning_joint>right_rear_wheel_joint</right_rear_wheel_spinning_joint>
+      <max_speed>20</max_speed>
+      <!-- 물리 파라미터 -->
       <wheel_separation>0.2413</wheel_separation>
-      <wheel_radius>0.0508</wheel_radius>
-      <wheel_torque>100</wheel_torque>
-      <wheel_acceleration>10.0</wheel_acceleration>
-      <command_topic>cmd_vel</command_topic>
+      <wheelbase>0.3302</wheelbase>
+      <wheel_diameter>0.1016</wheel_diameter>
+      <!-- 프레임 설정 -->
       <odometry_frame>odom</odometry_frame>
-      <odometry_topic>odom</odometry_topic>
       <robot_base_frame>base_link</robot_base_frame>
+      <!-- 출력 설정 -->
       <publish_odom>true</publish_odom>
-      <publish_wheel_tf>false</publish_wheel_tf>
-      <publish_odom_tf>true</publish_odom_tf>
-      <publish_wheel_joint_state>true</publish_wheel_joint_state>
-      <legacy_mode>false</legacy_mode>
+      <publish_odom_tf>true</publish_odom_tf>  <!-- Gazebo가 물리적으로 위치 결정 -->
+      <publish_wheel_tf>false</publish_wheel_tf>  <!-- robot_state_publisher가 담당 -->
+      <publish_wheel_joint_state>false</publish_wheel_joint_state>  <!-- robot_state_publisher가 담당 -->
     </plugin>
   </gazebo>

Commit message: 일단 스폰은 가능

File: f110_description/urdf/f1tenth.urdf.xacro (robot description, xacro)
@@ -21,4 +21,18 @@
   </material>
   <!-- ============================================ -->
+  <!-- Base Footprint (Dummy Root Link for KDL) -->
+  <!-- ============================================ -->
+  <!-- This is a dummy link with no inertia to satisfy KDL requirements -->
+  <link name="base_footprint">
+    <!-- No inertial, visual, or collision - just a reference frame -->
+  </link>
+  <!-- Fixed joint connecting base_footprint to base_link -->
+  <joint name="base_footprint_joint" type="fixed">
+    <parent link="base_footprint"/>
+    <child link="base_link"/>
+    <!-- base_link origin is at ground level, same as base_footprint -->
+    <origin xyz="0 0 0" rpy="0 0 0"/>
+  </joint>
+  <!-- ============================================ -->
   <!-- Base Link (Chassis) -->
   <!-- ============================================ -->
@@ -39,10 +53,4 @@
       <material name="blue"/>
     </visual>
-    <collision>
-      <origin xyz="0.165 0 0.09" rpy="0 0 0"/>
-      <geometry>
-        <box size="0.05 0.001 0.006"/>  <!-- Very small to avoid wheel collision -->
-      </geometry>
-    </collision>
   </link>
   <!-- ============================================ -->
@@ -346,46 +354,62 @@
     <self_collide>false</self_collide>
   </gazebo>
-  <!-- Ackermann Drive Controller Plugin -->
+  <!-- ============================================ -->
+  <!-- ros2_control Configuration -->
+  <!-- ============================================ -->
+  <ros2_control name="f1tenth_system" type="system">
+    <hardware>
+      <plugin>gazebo_ros2_control/GazeboSystem</plugin>
+    </hardware>
+    <!-- Rear Wheels (Traction/Drive) -->
+    <joint name="left_rear_wheel_joint">
+      <command_interface name="velocity">
+        <param name="min">-50</param>
+        <param name="max">50</param>
+      </command_interface>
+      <state_interface name="position"/>
+      <state_interface name="velocity"/>
+    </joint>
+    <joint name="right_rear_wheel_joint">
+      <command_interface name="velocity">
+        <param name="min">-50</param>
+        <param name="max">50</param>
+      </command_interface>
+      <state_interface name="position"/>
+      <state_interface name="velocity"/>
+    </joint>
+    <!-- Front Wheels (Passive rotation) -->
+    <joint name="left_front_wheel_joint">
+      <state_interface name="position"/>
+      <state_interface name="velocity"/>
+    </joint>
+    <joint name="right_front_wheel_joint">
+      <state_interface name="position"/>
+      <state_interface name="velocity"/>
+    </joint>
+    <!-- Steering Joints (Position control) -->
+    <joint name="left_steering_hinge_joint">
+      <command_interface name="position">
+        <param name="min">-0.4189</param>
+        <param name="max">0.4189</param>
+      </command_interface>
+      <state_interface name="position"/>
+      <state_interface name="velocity"/>
+    </joint>
+    <joint name="right_steering_hinge_joint">
+      <command_interface name="position">
+        <param name="min">-0.4189</param>
+        <param name="max">0.4189</param>
+      </command_interface>
+      <state_interface name="position"/>
+      <state_interface name="velocity"/>
+    </joint>
+  </ros2_control>
+  <!-- Gazebo ros2_control Plugin -->
   <gazebo>
-    <plugin name="gazebo_ros_ackermann_drive" filename="libgazebo_ros_ackermann_drive.so">
+    <plugin filename="libgazebo_ros2_control.so" name="gazebo_ros2_control">
       <ros>
-        <namespace>/f1tenth</namespace>
-        <remapping>cmd_vel:=cmd_vel</remapping>
-        <remapping>odom:=odom</remapping>
+        <namespace>/</namespace>
+        <remapping>/robot_description:=/robot_description</remapping>
       </ros>
-      <update_rate>100.0</update_rate>
-      <!-- 바퀴 조인트 (회전) -->
-      <front_left_joint>left_front_wheel_joint</front_left_joint>
-      <front_right_joint>right_front_wheel_joint</front_right_joint>
-      <rear_left_joint>left_rear_wheel_joint</rear_left_joint>
-      <rear_right_joint>right_rear_wheel_joint</rear_right_joint>
-      <!-- 조향 조인트 -->
-      <left_steering_joint>left_steering_hinge_joint</left_steering_joint>
-      <right_steering_joint>right_steering_hinge_joint</right_steering_joint>
-      <!-- 핵심: steering_wheel_joint 추가 (필수!) -->
-      <steering_wheel_joint>steering_wheel_joint</steering_wheel_joint>
-      <!-- PID Gains 추가 (안정성 향상) -->
-      <left_steering_pid_gain>1500 0 1</left_steering_pid_gain>
-      <left_steering_i_range>0 0</left_steering_i_range>
-      <right_steering_pid_gain>1500 0 1</right_steering_pid_gain>
-      <right_steering_i_range>0 0</right_steering_i_range>
-      <linear_velocity_pid_gain>1000 0 1</linear_velocity_pid_gain>
-      <linear_velocity_i_range>0 0</linear_velocity_i_range>
-      <!-- 조향 제한 -->
-      <max_steer>0.4189</max_steer>
-      <max_steering_angle>7.85</max_steering_angle>
-      <max_speed>20</max_speed>
-      <!-- 물리 파라미터 -->
-      <wheel_separation>0.2413</wheel_separation>
-      <wheelbase>0.3302</wheelbase>
-      <wheel_diameter>0.1016</wheel_diameter>
-      <!-- 프레임 설정 -->
-      <odometry_frame>odom</odometry_frame>
-      <robot_base_frame>base_link</robot_base_frame>
-      <!-- 출력 설정 -->
-      <publish_odom>true</publish_odom>
-      <publish_odom_tf>true</publish_odom_tf>  <!-- Gazebo가 물리적으로 위치 결정 -->
-      <publish_wheel_tf>false</publish_wheel_tf>  <!-- robot_state_publisher가 담당 -->
-      <publish_wheel_joint_state>false</publish_wheel_joint_state>  <!-- robot_state_publisher가 담당 -->
     </plugin>
   </gazebo>
