Commit message: 제어 가능?

File: f110_description/urdf/f1tenth.urdf.xacro (robot description, xacro)
@@ -21,20 +21,7 @@
   </material>
   <!-- ============================================ -->
-  <!-- Base Footprint (Dummy Root Link for KDL) -->
-  <!-- ============================================ -->
-  <!-- This is a dummy link with no inertia to satisfy KDL requirements -->
-  <link name="base_footprint">
-    <!-- No inertial, visual, or collision - just a reference frame -->
-  </link>
-  <!-- Fixed joint connecting base_footprint to base_link -->
-  <joint name="base_footprint_joint" type="fixed">
-    <parent link="base_footprint"/>
-    <child link="base_link"/>
-    <!-- base_link origin is at ground level, same as base_footprint -->
-    <origin xyz="0 0 0" rpy="0 0 0"/>
-  </joint>
-  <!-- ============================================ -->
-  <!-- Base Link (Chassis) -->
-  <!-- ============================================ -->
+  <!-- Base Link (Chassis) - Root Link -->
+  <!-- ============================================ -->
+  <!-- Note: KDL warning "root link has inertia" is harmless and can be ignored -->
   <link name="base_link">
     <inertial>
@@ -109,5 +96,5 @@
   </gazebo>
   <!-- ============================================ -->
-  <!-- Steering Wheel (dummy joint for Ackermann plugin) -->
+  <!-- Virtual Steering Wheel (Required by gazebo_ros_ackermann_drive) -->
   <!-- ============================================ -->
   <joint name="steering_wheel_joint" type="revolute">
@@ -116,5 +103,5 @@
     <origin xyz="0.15 0 0.25" rpy="0 0 0"/>
     <axis xyz="0 0 1"/>
-    <limit lower="-6.283" upper="6.283" effort="5.0" velocity="4.0"/>
+    <limit lower="-6.283" upper="6.283" effort="100.0" velocity="10.0"/>
   </joint>
   <link name="steering_wheel_link">
@@ -170,5 +157,5 @@
     <child link="right_rear_wheel"/>
     <origin xyz="0 -0.12065 0.0508" rpy="0 0 0"/>
-    <axis xyz="0 1 0"/>
+    <axis xyz="0 -1 0"/>
     <dynamics damping="0.1" friction="0.1"/>
   </joint>
@@ -208,6 +195,6 @@
     <origin xyz="0.3302 0.12065 0.0508" rpy="0 0 0"/>
     <axis xyz="0 0 1"/>  <!-- Steering axis (vertical) -->
-    <limit lower="-0.4189" upper="0.4189" effort="10.0" velocity="3.2"/>  <!-- ±24°, from F1TENTH Gym -->
-    <dynamics damping="0.7" friction="0.5"/>
+    <limit lower="-0.4189" upper="0.4189" effort="10.0" velocity="3.2"/>
+    <dynamics damping="0.7" friction="1.0"/>
   </joint>
   <link name="left_steering_hinge">
@@ -227,5 +214,5 @@
     <origin xyz="0 0 0" rpy="0 0 0"/>
     <axis xyz="0 1 0"/>
-    <dynamics damping="0.1" friction="0.1"/>
+    <dynamics damping="0.5" friction="1.0"/>
   </joint>
   <link name="left_front_wheel">
@@ -262,5 +249,5 @@
     <axis xyz="0 0 1"/>
     <limit lower="-0.4189" upper="0.4189" effort="10.0" velocity="3.2"/>
-    <dynamics damping="0.7" friction="0.5"/>
+    <dynamics damping="0.7" friction="1.0"/>
   </joint>
   <link name="right_steering_hinge">
@@ -279,6 +266,6 @@
     <child link="right_front_wheel"/>
     <origin xyz="0 0 0" rpy="0 0 0"/>
-    <axis xyz="0 1 0"/>
-    <dynamics damping="0.1" friction="0.1"/>
+    <axis xyz="0 -1 0"/>
+    <dynamics damping="0.5" friction="1.0"/>
   </joint>
   <link name="right_front_wheel">
@@ -324,5 +311,5 @@
     <kd>1.0</kd>
     <minDepth>0.005</minDepth>
-    <maxVel>0.1</maxVel>
+    <maxVel>100.0</maxVel>
     <self_collide>false</self_collide>
   </gazebo>
@@ -333,5 +320,5 @@
     <kd>1.0</kd>
     <minDepth>0.005</minDepth>
-    <maxVel>0.1</maxVel>
+    <maxVel>100.0</maxVel>
     <self_collide>false</self_collide>
   </gazebo>
@@ -342,5 +329,5 @@
     <kd>1.0</kd>
     <minDepth>0.005</minDepth>
-    <maxVel>0.1</maxVel>
+    <maxVel>100.0</maxVel>
     <self_collide>false</self_collide>
   </gazebo>
@@ -351,65 +338,48 @@
     <kd>1.0</kd>
     <minDepth>0.005</minDepth>
-    <maxVel>0.1</maxVel>
-    <self_collide>false</self_collide>
-  </gazebo>
-  <!-- ============================================ -->
-  <!-- ros2_control Configuration -->
-  <!-- ============================================ -->
-  <ros2_control name="f1tenth_system" type="system">
-    <hardware>
-      <plugin>gazebo_ros2_control/GazeboSystem</plugin>
-    </hardware>
-    <!-- Rear Wheels (Traction/Drive) -->
-    <joint name="left_rear_wheel_joint">
-      <command_interface name="velocity">
-        <param name="min">-50</param>
-        <param name="max">50</param>
-      </command_interface>
-      <state_interface name="position"/>
-      <state_interface name="velocity"/>
-    </joint>
-    <joint name="right_rear_wheel_joint">
-      <command_interface name="velocity">
-        <param name="min">-50</param>
-        <param name="max">50</param>
-      </command_interface>
-      <state_interface name="position"/>
-      <state_interface name="velocity"/>
-    </joint>
-    <!-- Front Wheels (Passive rotation) -->
-    <joint name="left_front_wheel_joint">
-      <state_interface name="position"/>
-      <state_interface name="velocity"/>
-    </joint>
-    <joint name="right_front_wheel_joint">
-      <state_interface name="position"/>
-      <state_interface name="velocity"/>
-    </joint>
-    <!-- Steering Joints (Position control) -->
-    <joint name="left_steering_hinge_joint">
-      <command_interface name="position">
-        <param name="min">-0.4189</param>
-        <param name="max">0.4189</param>
-      </command_interface>
-      <state_interface name="position"/>
-      <state_interface name="velocity"/>
-    </joint>
-    <joint name="right_steering_hinge_joint">
-      <command_interface name="position">
-        <param name="min">-0.4189</param>
-        <param name="max">0.4189</param>
-      </command_interface>
-      <state_interface name="position"/>
-      <state_interface name="velocity"/>
-    </joint>
-  </ros2_control>
-  <!-- Gazebo ros2_control Plugin -->
+    <maxVel>100.0</maxVel>
+    <self_collide>false</self_collide>
+  </gazebo>
+  <!-- ============================================ -->
+  <!-- Joint State Publisher Plugin -->
+  <!-- ============================================ -->
   <gazebo>
-    <plugin filename="libgazebo_ros2_control.so" name="gazebo_ros2_control">
+    <plugin name="gazebo_ros_joint_state_publisher" filename="libgazebo_ros_joint_state_publisher.so">
+      <update_rate>50</update_rate>
+      <joint_name>left_rear_wheel_joint</joint_name>
+      <joint_name>right_rear_wheel_joint</joint_name>
+      <joint_name>left_front_wheel_joint</joint_name>
+      <joint_name>right_front_wheel_joint</joint_name>
+      <joint_name>left_steering_hinge_joint</joint_name>
+      <joint_name>right_steering_hinge_joint</joint_name>
+    </plugin>
+  </gazebo>
+  <!-- ============================================ -->
+  <!-- F1TENTH Ackermann Drive Plugin -->
+  <!-- ============================================ -->
+  <gazebo>
+    <plugin name="f1tenth_drive_plugin" filename="libf1tenth_drive_plugin.so">
       <ros>
         <namespace>/</namespace>
-        <remapping>/robot_description:=/robot_description</remapping>
       </ros>
+      <!-- Update rate -->
+      <update_rate>100.0</update_rate>
+      <!-- Wheel joints -->
+      <front_left_wheel_joint>left_front_wheel_joint</front_left_wheel_joint>
+      <front_right_wheel_joint>right_front_wheel_joint</front_right_wheel_joint>
+      <rear_left_wheel_joint>left_rear_wheel_joint</rear_left_wheel_joint>
+      <rear_right_wheel_joint>right_rear_wheel_joint</rear_right_wheel_joint>
+      <!-- Steering joints -->
+      <front_left_steering_joint>left_steering_hinge_joint</front_left_steering_joint>
+      <front_right_steering_joint>right_steering_hinge_joint</front_right_steering_joint>
+      <!-- Vehicle parameters -->
+      <wheelbase>0.3302</wheelbase>
+      <track_width>0.2413</track_width>
+      <wheel_radius>0.0508</wheel_radius>
+      <!-- Steering limits -->
+      <max_steer_angle>0.4189</max_steer_angle>
+      <!-- Control parameters -->
+      <!-- Flip wheel rotation if measured sign is opposite (1.0 or -1.0) -->
+      <wheel_rotation_sign>-1.0</wheel_rotation_sign>
     </plugin>
   </gazebo>

Commit message: 제어 가능

File: f110_description/urdf/f1tenth.urdf.xacro (robot description, xacro)
@@ -157,5 +157,5 @@
     <child link="right_rear_wheel"/>
     <origin xyz="0 -0.12065 0.0508" rpy="0 0 0"/>
-    <axis xyz="0 -1 0"/>
+    <axis xyz="0 1 0"/>
     <dynamics damping="0.1" friction="0.1"/>
   </joint>
@@ -214,5 +214,5 @@
     <origin xyz="0 0 0" rpy="0 0 0"/>
     <axis xyz="0 1 0"/>
-    <dynamics damping="0.5" friction="1.0"/>
+    <dynamics damping="0.0" friction="0.0"/>
   </joint>
   <link name="left_front_wheel">
@@ -266,6 +266,6 @@
     <child link="right_front_wheel"/>
     <origin xyz="0 0 0" rpy="0 0 0"/>
-    <axis xyz="0 -1 0"/>
-    <dynamics damping="0.5" friction="1.0"/>
+    <axis xyz="0 1 0"/>
+    <dynamics damping="0.0" friction="0.0"/>
   </joint>
   <link name="right_front_wheel">

Commit message: 제어 가능! 및 자율주행 시스템 초안

File: f110_description/urdf/f1tenth.urdf.xacro (robot description, xacro)
@@ -1,14 +1,5 @@
 <?xml version="1.0"?>
-<!--
-F1TENTH Race Car URDF with Complete Physics Properties
-Based on: f1tenth_gym and f1tenth_gym_ros
-Vehicle: Traxxas Fiesta ST Rally 1/10 Scale
--->
 <robot name="f1tenth_racecar" xmlns:xacro="http://www.ros.org/wiki/xacro">
-  <!-- Include Hokuyo LiDAR -->
   <xacro:include filename="$(find f110_description)/urdf/hokuyo.urdf.xacro"/>
-  <!-- ============================================ -->
-  <!-- Materials -->
-  <!-- ============================================ -->
   <material name="black">
     <color rgba="0.2 0.2 0.2 1.0"/>
@@ -20,28 +11,21 @@
     <color rgba="0.8 0.0 0.0 1.0"/>
   </material>
-  <!-- ============================================ -->
-  <!-- Base Link (Chassis) - Root Link -->
-  <!-- ============================================ -->
-  <!-- Note: KDL warning "root link has inertia" is harmless and can be ignored -->
   <link name="base_link">
     <inertial>
+      <origin xyz="0.12 0 0.04" rpy="0 0 0"/>
+      <mass value="8.0"/>
+      <inertia
+        ixx="0.0730" ixy="0.0" ixz="0.0"
+        iyy="0.1093" iyz="0.0"
+        izz="0.0754"/>
+    </inertial>
+    <visual>
       <origin xyz="0.165 0 0.09" rpy="0 0 0"/>
-      <mass value="5.0"/>  <!-- F1TENTH mass from gym -->
-      <inertia
-        ixx="0.0456" ixy="0.0" ixz="0.0"
-        iyy="0.0683" iyz="0.0"
-        izz="0.04712"/> <!-- From f1tenth_gym parameters -->
-    </inertial>
-    <visual>
-      <origin xyz="0.165 0 0.09" rpy="0 0 0"/>
-      <geometry>
-        <box size="0.3302 0.2032 0.1"/>  <!-- wheelbase x width x height -->
+      <geometry>
+        <box size="0.3302 0.2032 0.1"/>
       </geometry>
       <material name="blue"/>
     </visual>
   </link>
-  <!-- ============================================ -->
-  <!-- LiDAR (Hokuyo 10LX) -->
-  <!-- ============================================ -->
   <xacro:hokuyo_10lx
     parent="base_link"
@@ -56,7 +40,4 @@
     <origin xyz="0.275 0 0.19" rpy="0 0 0"/>
   </xacro:hokuyo_10lx>
-  <!-- ============================================ -->
-  <!-- IMU Sensor -->
-  <!-- ============================================ -->
   <joint name="base_to_imu" type="fixed">
     <parent link="base_link"/>
@@ -81,5 +62,4 @@
     </collision>
   </link>
-  <!-- Gazebo IMU Sensor -->
   <gazebo reference="imu_link">
     <sensor name="imu_sensor" type="imu">
@@ -95,7 +75,4 @@
     </sensor>
   </gazebo>
-  <!-- ============================================ -->
-  <!-- Virtual Steering Wheel (Required by gazebo_ros_ackermann_drive) -->
-  <!-- ============================================ -->
   <joint name="steering_wheel_joint" type="revolute">
     <parent link="base_link"/>
@@ -115,23 +92,19 @@
     </inertial>
   </link>
-  <!-- ============================================ -->
-  <!-- Rear Wheels (Fixed, Motor Controlled) -->
-  <!-- ============================================ -->
-  <!-- Left Rear Wheel -->
   <joint name="left_rear_wheel_joint" type="continuous">
     <parent link="base_link"/>
     <child link="left_rear_wheel"/>
-    <origin xyz="0 0.12065 0.0508" rpy="0 0 0"/>  <!-- y = (wheel_width + width)/2 -->
-    <axis xyz="0 1 0"/>  <!-- Rotation around Y axis -->
-    <dynamics damping="0.1" friction="0.1"/>
+    <origin xyz="0 0.12065 0.0508" rpy="0 0 0"/>
+    <axis xyz="0 1 0"/>
+    <dynamics damping="0.1" friction="0.05"/>
   </joint>
   <link name="left_rear_wheel">
     <inertial>
-      <mass value="0.34055"/>  <!-- Wheel mass -->
+      <mass value="0.34055"/>
       <origin xyz="0 0 0" rpy="0 0 0"/>
       <inertia
         ixx="0.00026046" ixy="0.0" ixz="0.0"
         iyy="0.00026046" iyz="0.0"
-        izz="0.00044"/>  <!-- Cylinder inertia -->
+        izz="0.00044"/>
     </inertial>
     <visual>
@@ -140,5 +113,5 @@
       </geometry>
       <material name="black"/>
-      <origin xyz="0 0 0" rpy="1.5707963 0 0"/>  <!-- pi/2 rotation -->
+      <origin xyz="0 0 0" rpy="1.5707963 0 0"/>
     </visual>
     <collision>
@@ -152,5 +125,4 @@
     </collision>
   </link>
-  <!-- Right Rear Wheel -->
   <joint name="right_rear_wheel_joint" type="continuous">
     <parent link="base_link"/>
@@ -158,5 +130,5 @@
     <origin xyz="0 -0.12065 0.0508" rpy="0 0 0"/>
     <axis xyz="0 1 0"/>
-    <dynamics damping="0.1" friction="0.1"/>
+    <dynamics damping="0.1" friction="0.05"/>
   </joint>
   <link name="right_rear_wheel">
@@ -186,13 +158,9 @@
     </collision>
   </link>
-  <!-- ============================================ -->
-  <!-- Front Wheels (Steerable, Ackermann) -->
-  <!-- ============================================ -->
-  <!-- Left Front Steering Hinge -->
   <joint name="left_steering_hinge_joint" type="revolute">
     <parent link="base_link"/>
     <child link="left_steering_hinge"/>
     <origin xyz="0.3302 0.12065 0.0508" rpy="0 0 0"/>
-    <axis xyz="0 0 1"/>  <!-- Steering axis (vertical) -->
+    <axis xyz="0 0 1"/>
     <limit lower="-0.4189" upper="0.4189" effort="10.0" velocity="3.2"/>
     <dynamics damping="0.7" friction="1.0"/>
@@ -208,5 +176,4 @@
     </inertial>
   </link>
-  <!-- Left Front Wheel -->
   <joint name="left_front_wheel_joint" type="continuous">
     <parent link="left_steering_hinge"/>
@@ -214,5 +181,5 @@
     <origin xyz="0 0 0" rpy="0 0 0"/>
     <axis xyz="0 1 0"/>
-    <dynamics damping="0.0" friction="0.0"/>
+    <dynamics damping="0.05" friction="0.01"/>
   </joint>
   <link name="left_front_wheel">
@@ -242,5 +209,4 @@
     </collision>
   </link>
-  <!-- Right Front Steering Hinge -->
   <joint name="right_steering_hinge_joint" type="revolute">
     <parent link="base_link"/>
@@ -261,5 +227,4 @@
     </inertial>
   </link>
-  <!-- Right Front Wheel -->
   <joint name="right_front_wheel_joint" type="continuous">
     <parent link="right_steering_hinge"/>
@@ -267,5 +232,5 @@
     <origin xyz="0 0 0" rpy="0 0 0"/>
     <axis xyz="0 1 0"/>
-    <dynamics damping="0.0" friction="0.0"/>
+    <dynamics damping="0.05" friction="0.01"/>
   </joint>
   <link name="right_front_wheel">
@@ -295,5 +260,4 @@
     </collision>
   </link>
-  <!-- Friction and contact parameters for base_link -->
   <gazebo reference="base_link">
     <mu1>0.1</mu1>
@@ -304,83 +268,127 @@
     <self_collide>false</self_collide>
   </gazebo>
-  <!-- Friction parameters for wheels -->
   <gazebo reference="left_rear_wheel">
-    <mu1>1.5</mu1>
+    <mu1>1.0</mu1>
+    <mu2>1.0</mu2>
+    <kp>100000.0</kp>
+    <kd>10.0</kd>
+    <fdir1>1 0 0</fdir1>
+    <minDepth>0.001</minDepth>
+    <maxVel>10.0</maxVel>
+    <self_collide>false</self_collide>
+  </gazebo>
+  <gazebo reference="right_rear_wheel">
+    <mu1>1.0</mu1>
+    <mu2>1.0</mu2>
+    <kp>100000.0</kp>
+    <kd>10.0</kd>
+    <fdir1>1 0 0</fdir1>
+    <minDepth>0.001</minDepth>
+    <maxVel>10.0</maxVel>
+    <self_collide>false</self_collide>
+  </gazebo>
+  <gazebo reference="left_front_wheel">
+    <mu1>0.5</mu1>
     <mu2>1.5</mu2>
-    <kp>10000000.0</kp>
-    <kd>1.0</kd>
-    <minDepth>0.005</minDepth>
-    <maxVel>100.0</maxVel>
-    <self_collide>false</self_collide>
-  </gazebo>
-  <gazebo reference="right_rear_wheel">
-    <mu1>1.5</mu1>
+    <kp>100000.0</kp>
+    <kd>10.0</kd>
+    <fdir1>1 0 0</fdir1>
+    <minDepth>0.001</minDepth>
+    <maxVel>10.0</maxVel>
+    <self_collide>false</self_collide>
+  </gazebo>
+  <gazebo reference="right_front_wheel">
+    <mu1>0.5</mu1>
     <mu2>1.5</mu2>
-    <kp>10000000.0</kp>
-    <kd>1.0</kd>
-    <minDepth>0.005</minDepth>
-    <maxVel>100.0</maxVel>
-    <self_collide>false</self_collide>
-  </gazebo>
-  <gazebo reference="left_front_wheel">
-    <mu1>1.5</mu1>
-    <mu2>1.5</mu2>
-    <kp>10000000.0</kp>
-    <kd>1.0</kd>
-    <minDepth>0.005</minDepth>
-    <maxVel>100.0</maxVel>
-    <self_collide>false</self_collide>
-  </gazebo>
-  <gazebo reference="right_front_wheel">
-    <mu1>1.5</mu1>
-    <mu2>1.5</mu2>
-    <kp>10000000.0</kp>
-    <kd>1.0</kd>
-    <minDepth>0.005</minDepth>
-    <maxVel>100.0</maxVel>
-    <self_collide>false</self_collide>
-  </gazebo>
-  <!-- ============================================ -->
-  <!-- Joint State Publisher Plugin -->
-  <!-- ============================================ -->
+    <kp>100000.0</kp>
+    <kd>10.0</kd>
+    <fdir1>1 0 0</fdir1>
+    <minDepth>0.001</minDepth>
+    <maxVel>10.0</maxVel>
+    <self_collide>false</self_collide>
+  </gazebo>
+  <ros2_control name="f1tenth_system" type="system">
+    <hardware>
+      <plugin>gazebo_ros2_control/GazeboSystem</plugin>
+    </hardware>
+    <joint name="left_rear_wheel_joint">
+      <command_interface name="velocity">
+        <param name="min">-100.0</param>
+        <param name="max">100.0</param>
+      </command_interface>
+      <state_interface name="position"/>
+      <state_interface name="velocity"/>
+    </joint>
+    <joint name="right_rear_wheel_joint">
+      <command_interface name="velocity">
+        <param name="min">-100.0</param>
+        <param name="max">100.0</param>
+      </command_interface>
+      <state_interface name="position"/>
+      <state_interface name="velocity"/>
+    </joint>
+    <joint name="left_steering_hinge_joint">
+      <command_interface name="position">
+        <param name="min">-0.7</param>
+        <param name="max">0.7</param>
+      </command_interface>
+      <state_interface name="position"/>
+      <state_interface name="velocity"/>
+    </joint>
+    <joint name="right_steering_hinge_joint">
+      <command_interface name="position">
+        <param name="min">-0.7</param>
+        <param name="max">0.7</param>
+      </command_interface>
+      <state_interface name="position"/>
+      <state_interface name="velocity"/>
+    </joint>
+  </ros2_control>
   <gazebo>
-    <plugin name="gazebo_ros_joint_state_publisher" filename="libgazebo_ros_joint_state_publisher.so">
-      <update_rate>50</update_rate>
-      <joint_name>left_rear_wheel_joint</joint_name>
-      <joint_name>right_rear_wheel_joint</joint_name>
-      <joint_name>left_front_wheel_joint</joint_name>
-      <joint_name>right_front_wheel_joint</joint_name>
-      <joint_name>left_steering_hinge_joint</joint_name>
-      <joint_name>right_steering_hinge_joint</joint_name>
+    <plugin name="gazebo_ros2_control" filename="libgazebo_ros2_control.so">
+        <robot_param>robot_description</robot_param>
+        <robot_param_node>robot_state_publisher</robot_param_node>
+        <parameters>$(find f110_description)/config/ros2_control.yaml</parameters>
     </plugin>
   </gazebo>
-  <!-- ============================================ -->
-  <!-- F1TENTH Ackermann Drive Plugin -->
-  <!-- ============================================ -->
-  <gazebo>
-    <plugin name="f1tenth_drive_plugin" filename="libf1tenth_drive_plugin.so">
-      <ros>
-        <namespace>/</namespace>
-      </ros>
-      <!-- Update rate -->
-      <update_rate>100.0</update_rate>
-      <!-- Wheel joints -->
-      <front_left_wheel_joint>left_front_wheel_joint</front_left_wheel_joint>
-      <front_right_wheel_joint>right_front_wheel_joint</front_right_wheel_joint>
-      <rear_left_wheel_joint>left_rear_wheel_joint</rear_left_wheel_joint>
-      <rear_right_wheel_joint>right_rear_wheel_joint</rear_right_wheel_joint>
-      <!-- Steering joints -->
-      <front_left_steering_joint>left_steering_hinge_joint</front_left_steering_joint>
-      <front_right_steering_joint>right_steering_hinge_joint</front_right_steering_joint>
-      <!-- Vehicle parameters -->
-      <wheelbase>0.3302</wheelbase>
-      <track_width>0.2413</track_width>
-      <wheel_radius>0.0508</wheel_radius>
-      <!-- Steering limits -->
-      <max_steer_angle>0.4189</max_steer_angle>
-      <!-- Control parameters -->
-      <!-- Flip wheel rotation if measured sign is opposite (1.0 or -1.0) -->
-      <wheel_rotation_sign>-1.0</wheel_rotation_sign>
-    </plugin>
-  </gazebo>
+  <transmission name="left_rear_wheel_transmission">
+    <type>transmission_interface/SimpleTransmission</type>
+    <joint name="left_rear_wheel_joint">
+      <hardwareInterface>velocity</hardwareInterface>
+    </joint>
+    <actuator name="left_rear_wheel_actuator">
+      <hardwareInterface>velocity</hardwareInterface>
+      <mechanicalReduction>1</mechanicalReduction>
+    </actuator>
+  </transmission>
+  <transmission name="right_rear_wheel_transmission">
+    <type>transmission_interface/SimpleTransmission</type>
+    <joint name="right_rear_wheel_joint">
+      <hardwareInterface>velocity</hardwareInterface>
+    </joint>
+    <actuator name="right_rear_wheel_actuator">
+      <hardwareInterface>velocity</hardwareInterface>
+      <mechanicalReduction>1</mechanicalReduction>
+    </actuator>
+  </transmission>
+  <transmission name="left_steering_hinge_transmission">
+    <type>transmission_interface/SimpleTransmission</type>
+    <joint name="left_steering_hinge_joint">
+      <hardwareInterface>position</hardwareInterface>
+    </joint>
+    <actuator name="left_steering_hinge_actuator">
+      <hardwareInterface>position</hardwareInterface>
+      <mechanicalReduction>1</mechanicalReduction>
+    </actuator>
+  </transmission>
+  <transmission name="right_steering_hinge_transmission">
+    <type>transmission_interface/SimpleTransmission</type>
+    <joint name="right_steering_hinge_joint">
+      <hardwareInterface>position</hardwareInterface>
+    </joint>
+    <actuator name="right_steering_hinge_actuator">
+      <hardwareInterface>position</hardwareInterface>
+      <mechanicalReduction>1</mechanicalReduction>
+    </actuator>
+  </transmission>
 </robot>
